Commit message: Add painter class for drawing json

File: conf/vander_bot_v2.urdf (robot description, URDF)
Before this commit: robot painter, 4 links, 3 joints
Joints:
- joint base_link_link_01: axis 0 0 1 -> 0 0 -1; origin xyz=0 0 0.005 rpy=0 0 0.7853981633974483 -> xyz=0 0 0.005 rpy=0 0 0
- joint link_01_link_02: axis 0 0 1 -> 0 0 -1; origin xyz=0 0.3566 0.01 rpy=0 0 0 -> xyz=0.02467 0.35571 0.01 rpy=0 0 0
- joint link_02_tool: origin xyz=0 0.2896 0.0 rpy=0 0 0 -> xyz=0.02754 0.28 0.0 rpy=0 0 0
